File: Hardware Sumo/Sumo 2026.kicad_pcb (KiCad board)
At the start: 2 copper layers, 80 x 40 mm, 47 parts, among them J1 Conn_01x04_Pin, J10 Conn_01x03_Pin, J11 Conn_01x03_Pin, J12 Conn_01x03_Pin, J13 Conn_01x03_Pin, J14 Conn_01x04_Pin, J2 Conn_01x04_Pin, J3 DISPLAY, J4 Conn_01x03_Pin, J6 Conn_01x03_Pin, J7 Conn_01x03_Pin, J8 Conn_01x03_Pin, J9 Conn_01x03_Pin, SW1 SW_Push_Dual_x2, SW5 SW_Push_Dual_x2, SW6 SW_Push_Dual_x2, U1 AMS1117-3.3, U3 ESP32-WROOM-32

Commit message: Add files via upload
Parts:
- added J5: Conn_01x02_Pin, Connector_JST:JST_XH_B2B-XH-A_1x02_P2.50mm_Vertical, F.Cu at (118.1, 67.0)
Connections:
- U3 pad 5: /SW2 -> /R
- U3 pad 6: /SW1 -> unconnected-(U3-IO34-Pad6)
- U3 pad 7: unconnected-(U3-IO35-Pad7) -> /SW2
- U3 pad 8: unconnected-(U3-IO32-Pad8) -> /SW1
Routing:
- net /R: track 0.00 -> 39.1 mm, vias 0 -> 1
- net /SW1: track 31.8 -> 30.7 mm
- net /EN: track 56.6 -> 56.0 mm
